Commit message: update

File: src/orbit_robot_description/urdf/fairino10_v6.urdf (robot description, URDF)
Before this commit: robot fairino10_v6_robot, 7 links, 6 joints
Links:
- added link world
- link base_link: geometry collision mesh filename=file:///home/sam/orbit_sim_ws/src/orbit_robot_description/m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; visual mesh filename=file:///home/sam/orbit_sim_ws/src/orbit_robot_description/m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
- link forearm_link: geometry collision mesh filename=file:///home/sam/orbit_sim_ws/src/orbit_robot_description/m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; visual mesh filename=file:///home/sam/orbit_sim_ws/src/orbit_robot_description/m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
- link shoulder_link: geometry collision mesh filename=file:///home/sam/orbit_sim_ws/src/orbit_robot_description/m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; visual mesh filename=file:///home/sam/orbit_sim_ws/src/orbit_robot_description/m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
- link upperarm_link: geometry collision mesh filename=file:///home/sam/orbit_sim_ws/src/orbit_robot_description/m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; visual mesh filename=file:///home/sam/orbit_sim_ws/src/orbit_robot_description/m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
- link wrist1_link: geometry collision mesh filename=file:///home/sam/orbit_sim_ws/src/orbit_robot_description/m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; visual mesh filename=file:///home/sam/orbit_sim_ws/src/orbit_robot_description/m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
- link wrist2_link: geometry collision mesh filename=file:///home/sam/orbit_sim_ws/src/orbit_robot_description/m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; visual mesh filename=file:///home/sam/orbit_sim_ws/src/orbit_robot_description/m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
- link wrist3_link: geometry collision mesh filename=file:///home/sam/orbit_sim_ws/src/orbit_robot_description/m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; visual mesh filename=file:///home/sam/orbit_sim_ws/src/orbit_robot_description/m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
Joints:
- added joint world_joint: type fixed, parent world, child base_link, origin xyz=0.0 0.0 0.0 rpy=0 0 0
